File: BenchBudEE/PowerAdjustmentMonitor.sch (KiCad schematic (older format))
At the start: 15 parts, among them U6 LM317, U7 LM317, U8 7805, U9 7805

Commit message: Associating and Placing the Power Modification Module
Parts:
- removed JP2, JP3: JUMPER, ~, symbol JUMPER
- removed U6: LM317, ~, symbol LM317
- removed U8, U9: 7805, ~, symbol 7805
- added C14, C15, C16, C17, C18, C19, C20, C21, C22, C23, C24, C25: C, ~, symbol C
- added D10, D11, D12, D13, D6, D7, D8, D9: MMBD914-7-F, ~, symbol DIODE
- added R52, R53, R54, R55: R, ~, symbol R
- added U6, U9: LM337T, TO-220, symbol LM337T
- added U8: LM317, ~, symbol LM317
- R34, R37: value R -> 715
- R35, R36: value RVAR -> 5k
Connections:
- wire segments 56 -> 102
Other:
- note added: "-1.5 to -10V Output"
- note added: "-10V output"
- note added: "1.5 to 10V Output"
- note added: "10V output"
- moved on the sheet: R36, R37, R40, R41
