File: BenchBudEE/PowerAdjustmentMonitor.sch (KiCad schematic (older format))
At the start: 37 parts, among them U6 LM337T, U7 LM317, U8 LM317, U9 LM337T

Commit message: Layout Work Session 4
Parts:
- removed JP1: JUMPER, ~, symbol JUMPER
Connections:
- net labels added: GND_PWR, GND_TC
- net labels removed: AGND, GND
- wire segments 102 -> 99
Other:
- moved on the sheet: C14, C15, C16, C17, C18, C19, C20, C21, C22, C23, C24, C25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

Commit message: Layout Work Session 5
Connections:
- net labels added: AGND
- net labels removed: GND_TC
- wire segments 99 -> 100
Changed lines of the file:
@@
 $EndDescr
 $Comp
-L +3.3V #PWR041
+L +3.3V #PWR042
 U 1 1 52F67086
 P 5550 5850
-F 0 "#PWR041" H 5550 5810 30  0001 C CNN
+F 0 "#PWR042" H 5550 5810 30  0001 C CNN
 F 1 "+3.3V" H 5550 5960 30  0000 C CNN
 F 2 "" H 5550 5850 60  0000 C CNN
@@
 $EndComp
 $Comp
-L +5V #PWR042
+L +5V #PWR043
 U 1 1 52F6708C
 P 5350 5850
-F 0 "#PWR042" H 5350 5940 20  0001 C CNN
+F 0 "#PWR043" H 5350 5940 20  0001 C CNN
 F 1 "+5V" H 5350 5940 30  0000 C CNN
 F 2 "" H 5350 5850 60  0000 C CNN
@@
 $EndComp
 $Comp
-L +12V #PWR043
+L +12V #PWR044
 U 1 1 52F67112
 P 6350 1700
-F 0 "#PWR043" H 6350 1650 20  0001 C CNN
+F 0 "#PWR044" H 6350 1650 20  0001 C CNN
 F 1 "+12V" H 6350 1800 30  0000 C CNN
 F 2 "" H 6350 1700 60  0000 C CNN
@@
 $EndComp
 $Comp
-L -12V #PWR044
+L -12V #PWR045
 U 1 1 52F67118
 P 1950 4950
-F 0 "#PWR044" H 1950 5080 20  0001 C CNN
+F 0 "#PWR045" H 1950 5080 20  0001 C CNN
 F 1 "-12V" H 1950 5050 30  0000 C CNN
 F 2 "" H 1950 4950 60  0000 C CNN
@@
 $EndComp
 $Comp
-L FE_V+ #PWR045
+L FE_V+ #PWR046
 U 1 1 52F672AE
 P 4500 2250
-F 0 "#PWR045" H 4500 2350 30  0001 C CNN
+F 0 "#PWR046" H 4500 2350 30  0001 C CNN
 F 1 "FE_V+" H 4500 2350 30  0000 C CNN
 F 2 "" H 4500 2250 60  0000 C CNN
@@
 F 3 "~" H 7700 3800 60  0000 C CNN
 	1    7700 3800
-	1    0    0    -1
+	-1   0    0    1
 $EndComp
 $Comp
@@
 	-1   0    0    1
 $EndComp
-Wire Wire Line
-	7700 3500 7700 3550
 Connection ~ 7700 4700
 Wire Wire Line
@@
 Wire Wire Line
 	6650 4050 6650 3500
-Connection ~ 7700 3500
 Wire Wire Line
 	3150 3500 3150 3900
@@
 Connection ~ 3700 3500
 $Comp
-L GND_PWR #PWR046
+L GND_PWR #PWR047
 U 1 1 53133BD8
 P 8600 3550
-F 0 "#PWR046" H 8600 3550 30  0001 C CNN
+F 0 "#PWR047" H 8600 3550 30  0001 C CNN
 F 1 "GND_PWR" H 8600 3480 30  0000 C CNN
 F 2 "" H 8600 3550 60  0000 C CNN
@@
 $EndComp
 $Comp
-L +12V #PWR047
+L +12V #PWR048
 U 1 1 53133BF5
 P 1950 2200
-F 0 "#PWR047" H 1950 2150 20  0001 C CNN
+F 0 "#PWR048" H 1950 2150 20  0001 C CNN
 F 1 "+12V" H 1950 2300 30  0000 C CNN
 F 2 "" H 1950 2200 60  0000 C CNN
@@
 	1950 2250 1950 2200
 $Comp
-L -12V #PWR048
+L -12V #PWR049
 U 1 1 53133CCE
 P 6300 4650
-F 0 "#PWR048" H 6300 4780 20  0001 C CNN
+F 0 "#PWR049" H 6300 4780 20  0001 C CNN
 F 1 "-12V" H 6300 4750 30  0000 C CNN
 F 2 "" H 6300 4650 60  0000 C CNN
@@
 Wire Wire Line
 	6300 4650 6300 4700
-$Comp
-L GND_TC #PWR049
-U 1 1 53133EDC
-P 2250 3600
-F 0 "#PWR049" H 2250 3600 30  0001 C CNN
-F 1 "GND_TC" H 2250 3530 30  0000 C CNN
-F 2 "" H 2250 3600 60  0000 C CNN
-F 3 "" H 2250 3600 60  0000 C CNN
-	1    2250 3600
-	1    0    0    -1
-$EndComp
 Wire Wire Line
 	2250 3500 4200 3500
@@
 Connection ~ 8250 3500
 Connection ~ 8600 3300
+$Comp
+L AGND #PWR050
+U 1 1 53138379
+P 2250 3600
+F 0 "#PWR050" H 2250 3600 40  0001 C CNN
+F 1 "AGND" H 2250 3530 50  0000 C CNN
+F 2 "" H 2250 3600 60  0000 C CNN
+F 3 "" H 2250 3600 60  0000 C CNN
+	1    2250 3600
+	1    0    0    -1
+$EndComp
+Wire Wire Line
+	7700 3050 7700 3100
+Wire Wire Line
+	7700 3550 7700 3500
+Connection ~ 7700 3500
 $EndSCHEMATC
