File: BenchBudEE/BenchBudEE.kicad_pcb (KiCad board)
At the start: 4 copper layers, 165.1 x 63.5 mm, 129 parts, among them K1 1461069-5, P1 24 pin Mini-fit Jr, P2 CONN_3X2, P3 CONN_2, P4 12 pin terminal block, P5 3 Pin TB, Q1 2N3904, Q2 DMN65D8L-7, Q3 B130-13-F, Q4 B130-13-F, SW1 Power Switch, U1 LTV-816S, U10 MCP4801, U2 MCP3901, U3 LMT84, U4 OPA4170, U5 AP5726, U6 LM337T, U7 LM317, U8 LM317, U9 LM337T

Commit message: Layout Work Session 6
Parts:
- added JP1: JUMPER, PIN_ARRAY_2X1, F.Cu at (166.0, 131.4)
- added JP2: JUMPER, PIN_ARRAY_2X1, F.Cu at (158.9, 128.8)
- added JP3: JUMPER, PIN_ARRAY_2X1, F.Cu at (166.0, 135.8)
- added JP4: JUMPER, PIN_ARRAY_2X1, F.Cu at (158.9, 138.9)
- C10, C11, D10, D11, D12, D13, D6, D7, D8, D9: moved to B.Cu
- R34, R37: moved to F.Cu
- moved C13 187.1 mm to (146.2, 151.5)
- moved C17 93.9 mm to (276.6, 109.5), turned to 180 degrees
- moved D9 91.4 mm to (275.1, 113.2)
- moved C20 86.9 mm to (263.7, 103.4)
- moved R54 83.7 mm to (269.2, 104.8), turned to 0 degrees
- moved R55 82.7 mm to (269.2, 107.1), turned to 180 degrees
- moved R52 81.7 mm to (259.6, 113.7), turned to 180 degrees
- moved C14 81.5 mm to (272.5, 101.5)
- moved D13 78.2 mm to (269.1, 113.5), turned to 180 degrees
- moved C19 77.5 mm to (245.0, 115.3)
- moved C6 76.6 mm to (236.9, 113.5), turned to 180 degrees
- moved D8 76.3 mm to (257.6, 107.2), turned to 90 degrees
- moved R49 74.9 mm to (241.3, 115.3)
- moved C24 74.5 mm to (272.0, 106.2), turned to 270 degrees
- moved R38 72.8 mm to (243.2, 111.4)
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Routing:
- net +3.3V: track 0.00 -> 151.2 mm
- net N-00000125: track 0.00 -> 52.2 mm
- net N-0000094: track 0.00 -> 49.4 mm
- net +12P: track 1.97 -> 47.8 mm, vias 1 -> 2
- net GND: track 0.00 -> 37.6 mm
- net -12P: track 0.00 -> 31.2 mm, vias 0 -> 1
- net N-00000104: track 0.00 -> 18.9 mm
- net /PowerAdjustmentMonitor/V-_ADJ: track 0.00 -> 16.8 mm
- net N-00000127: track 0.00 -> 9.84 mm
- net +5V: track 2.61 -> 11.0 mm, vias 1 -> 2
- net +5P: track 2.24 -> 10.5 mm, vias 1 -> 2
- net N-00000116: track 0.00 -> 6.76 mm
- added copper zone on GND, net GND
