File: BenchBudEE/Thermocouple.sch (KiCad schematic (older format))
At the start: 22 parts, among them P2 CONN_3X2, P3 CONN_2, U2 MCP3901, U3 LMT84, U4 OPA4170

Commit message: Layout Work Session 11
Parts:
- added L5: INDUCTOR, ~, symbol INDUCTOR
Connections:
- net +5V: now also L5.2; no longer C7.2, U2.2 (DVdd)
- new net: C7.2, L5.1, U2.2 (DVdd)
Other:
- moved on the sheet: C7
Changed lines of the file:
@@
 Sheet 2 9
 Title ""
-Date "3 mar 2014"
+Date "13 mar 2014"
 Rev ""
 Comp ""
@@
 $EndComp
 $Comp
-L +5V #PWR9
+L +5V #PWR8
 U 1 1 5303ACCB
 P 5800 4800
-F 0 "#PWR9" H 5800 4890 20  0001 C CNN
+F 0 "#PWR8" H 5800 4890 20  0001 C CNN
 F 1 "+5V" H 5800 4890 30  0000 C CNN
 F 2 "" H 5800 4800 60  0000 C CNN
@@
 $EndComp
 $Comp
-L +5V #PWR4
+L +5V #PWR3
 U 1 1 5303B53D
 P 3200 1550
-F 0 "#PWR4" H 3200 1640 20  0001 C CNN
+F 0 "#PWR3" H 3200 1640 20  0001 C CNN
 F 1 "+5V" H 3200 1640 30  0000 C CNN
 F 2 "" H 3200 1550 60  0000 C CNN
@@
 L C C7
 U 1 1 5303B7CA
-P 2350 1700
-F 0 "C7" H 2350 1800 40  0000 L CNN
-F 1 "C" H 2356 1615 40  0000 L CNN
-F 2 "~" H 2388 1550 30  0000 C CNN
-F 3 "~" H 2350 1700 60  0000 C CNN
-	1    2350 1700
-	0    -1   -1   0
-$EndComp
-$Comp
-L +5V #PWR2
-U 1 1 5303BA92
-P 2650 1550
-F 0 "#PWR2" H 2650 1640 20  0001 C CNN
-F 1 "+5V" H 2650 1640 30  0000 C CNN
-F 2 "" H 2650 1550 60  0000 C CNN
-F 3 "" H 2650 1550 60  0000 C CNN
-	1    2650 1550
-	1    0    0    -1
+P 2100 1700
+F 0 "C7" H 2100 1800 40  0000 L CNN
+F 1 "C" H 2106 1615 40  0000 L CNN
+F 2 "~" H 2138 1550 30  0000 C CNN
+F 3 "~" H 2100 1700 60  0000 C CNN
+	1    2100 1700
+	0    -1   -1   0
 $EndComp
 Text Notes 6550 5650 0    60   ~ 0
@@
 	3850 1700 3850 1800
 Wire Wire Line
-	2650 1550 2650 1900
-Wire Wire Line
-	2650 1700 2550 1700
-Connection ~ 2650 1700
-Wire Wire Line
 	2650 4250 2650 4550
 Wire Wire Line
 	3200 4250 3200 4550
-Wire Wire Line
-	2150 1700 1950 1700
-Wire Wire Line
-	1950 1700 1950 1800
 Wire Wire Line
 	1050 3150 1600 3150
@@
 MISO
 $Comp
-L FE_V+ #PWR13
+L FE_V+ #PWR12
 U 1 1 5311A08F
 P 6750 3650
-F 0 "#PWR13" H 6750 3750 30  0001 C CNN
+F 0 "#PWR12" H 6750 3750 30  0001 C CNN
 F 1 "FE_V+" H 6750 3750 30  0000 C CNN
 F 2 "" H 6750 3650 60  0000 C CNN
@@
 $EndComp
 $Comp
-L FE_V+ #PWR17
+L FE_V+ #PWR16
 U 1 1 5311A095
 P 9200 4900
-F 0 "#PWR17" H 9200 5000 30  0001 C CNN
+F 0 "#PWR16" H 9200 5000 30  0001 C CNN
 F 1 "FE_V+" H 9200 5000 30  0000 C CNN
 F 2 "" H 9200 4900 60  0000 C CNN
@@
 $EndComp
 $Comp
-L FE_V+ #PWR14
+L FE_V+ #PWR13
 U 1 1 5311A09B
 P 9200 1700
-F 0 "#PWR14" H 9200 1800 30  0001 C CNN
+F 0 "#PWR13" H 9200 1800 30  0001 C CNN
 F 1 "FE_V+" H 9200 1800 30  0000 C CNN
 F 2 "" H 9200 1700 60  0000 C CNN
@@
 $EndComp
 $Comp
-L FE_V- #PWR16
+L FE_V- #PWR15
 U 1 1 5311A0A1
 P 9200 3900
-F 0 "#PWR16" H 9200 4100 40  0001 C CNN
+F 0 "#PWR15" H 9200 4100 40  0001 C CNN
 F 1 "FE_V-" H 9200 4050 40  0000 C CNN
 F 2 "~" H 9200 3900 60  0000 C CNN
@@
 $EndComp
 $Comp
-L FE_V- #PWR15
+L FE_V- #PWR14
 U 1 1 5311A0A7
 P 9200 2700
-F 0 "#PWR15" H 9200 2900 40  0001 C CNN
+F 0 "#PWR14" H 9200 2900 40  0001 C CNN
 F 1 "FE_V-" H 9200 2850 40  0000 C CNN
 F 2 "~" H 9200 2700 60  0000 C CNN
@@
 $EndComp
 $Comp
-L FE_V- #PWR12
+L FE_V- #PWR11
 U 1 1 5311A0AD
 P 6750 2600
-F 0 "#PWR12" H 6750 2800 40  0001 C CNN
+F 0 "#PWR11" H 6750 2800 40  0001 C CNN
 F 1 "FE_V-" H 6750 2750 40  0000 C CNN
 F 2 "~" H 6750 2600 60  0000 C CNN
@@
 $EndComp
 $Comp
-L AGND #PWR3
+L AGND #PWR2
 U 1 1 5313730A
 P 2650 4550
-F 0 "#PWR3" H 2650 4550 40  0001 C CNN
+F 0 "#PWR2" H 2650 4550 40  0001 C CNN
 F 1 "AGND" H 2650 4480 50  0000 C CNN
 F 2 "" H 2650 4550 60  0000 C CNN
@@
 $EndComp
 $Comp
-L AGND #PWR5
+L AGND #PWR4
 U 1 1 53137321
 P 3200 4550
-F 0 "#PWR5" H 3200 4550 40  0001 C CNN
+F 0 "#PWR4" H 3200 4550 40  0001 C CNN
 F 1 "AGND" H 3200 4480 50  0000 C CNN
 F 2 "" H 3200 4550 60  0000 C CNN
@@
 L AGND #PWR1
 U 1 1 5313732C
-P 1950 1800
-F 0 "#PWR1" H 1950 1800 40  0001 C CNN
-F 1 "AGND" H 1950 1730 50  0000 C CNN
-F 2 "" H 1950 1800 60  0000 C CNN
-F 3 "" H 1950 1800 60  0000 C CNN
-	1    1950 1800
-	1    0    0    -1
-$EndComp
-$Comp
-L AGND #PWR6
+P 1700 1800
+F 0 "#PWR1" H 1700 1800 40  0001 C CNN
+F 1 "AGND" H 1700 1730 50  0000 C CNN
+F 2 "" H 1700 1800 60  0000 C CNN
+F 3 "" H 1700 1800 60  0000 C CNN
+	1    1700 1800
+	1    0    0    -1
+$EndComp
+$Comp
+L AGND #PWR5
 U 1 1 5313733C
 P 3850 1800
-F 0 "#PWR6" H 3850 1800 40  0001 C CNN
+F 0 "#PWR5" H 3850 1800 40  0001 C CNN
 F 1 "AGND" H 3850 1730 50  0000 C CNN
 F 2 "" H 3850 1800 60  0000 C CNN
@@
 $EndComp
 $Comp
-L AGND #PWR10
+L AGND #PWR9
 U 1 1 53137342
 P 6050 2750
-F 0 "#PWR10" H 6050 2750 40  0001 C CNN
+F 0 "#PWR9" H 6050 2750 40  0001 C CNN
 F 1 "AGND" H 6050 2680 50  0000 C CNN
 F 2 "" H 6050 2750 60  0000 C CNN
@@
 $EndComp
 $Comp
-L AGND #PWR11
+L AGND #PWR10
 U 1 1 53137352
 P 6050 3700
-F 0 "#PWR11" H 6050 3700 40  0001 C CNN
+F 0 "#PWR10" H 6050 3700 40  0001 C CNN
 F 1 "AGND" H 6050 3630 50  0000 C CNN
 F 2 "" H 6050 3700 60  0000 C CNN
@@
 $EndComp
 $Comp
-L AGND #PWR7
+L AGND #PWR6
 U 1 1 53137362
 P 5250 4550
-F 0 "#PWR7" H 5250 4550 40  0001 C CNN
+F 0 "#PWR6" H 5250 4550 40  0001 C CNN
 F 1 "AGND" H 5250 4480 50  0000 C CNN
 F 2 "" H 5250 4550 60  0000 C CNN
@@
 $EndComp
 $Comp
-L AGND #PWR8
+L AGND #PWR7
 U 1 1 53137372
 P 5250 6650
-F 0 "#PWR8" H 5250 6650 40  0001 C CNN
+F 0 "#PWR7" H 5250 6650 40  0001 C CNN
 F 1 "AGND" H 5250 6580 50  0000 C CNN
 F 2 "" H 5250 6650 60  0000 C CNN
@@
 	1    0    0    -1
 $EndComp
+$Comp
+L INDUCTOR L5
+U 1 1 5321FEC1
+P 2850 1750
+F 0 "L5" V 2800 1750 40  0000 C CNN
+F 1 "INDUCTOR" V 2950 1750 40  0000 C CNN
+F 2 "~" H 2850 1750 60  0000 C CNN
+F 3 "~" H 2850 1750 60  0000 C CNN
+	1    2850 1750
+	0    -1   -1   0
+$EndComp
+Wire Wire Line
+	2650 1900 2650 1850
+Wire Wire Line
+	2650 1850 2550 1850
+Wire Wire Line
+	2550 1850 2550 1700
+Wire Wire Line
+	2550 1700 2300 1700
+Connection ~ 2550 1750
+Wire Wire Line
+	1900 1700 1700 1700
+Wire Wire Line
+	1700 1700 1700 1800
+Wire Wire Line
+	3150 1750 3200 1750
+Connection ~ 3200 1750
 $EndSCHEMATC
