File: BenchBudEE/Thermocouple.sch (KiCad schematic (older format))
At the start: 23 parts, among them P2 CONN_3X2, P3 CONN_2, U2 MCP3901, U3 LMT84, U4 OPA4170

Commit message: Layout Work Session 14
Parts:
- added C30, C31: C, SM0805, symbol C
Connections:
- net REF- is gone; now on net AGND: U2.10 (REFIN-)
- net AGND: now also C31.2
- net at U2.15 (OSC1): now also C30.1
- net at U2.16 (OSC2): now also C30.2
- net REF+: no longer names the net of U2.9 (REFIN/OUT+)
- net REF+: now also C31.1
Changed lines of the file:
@@
 Sheet 2 9
 Title ""
-Date "15 mar 2014"
+Date "16 mar 2014"
 Rev ""
 Comp ""
@@
 $EndComp
 $Comp
-L +5V #PWR8
+L +5V #PWR9
 U 1 1 5303ACCB
 P 5800 4800
-F 0 "#PWR8" H 5800 4890 20  0001 C CNN
+F 0 "#PWR9" H 5800 4890 20  0001 C CNN
 F 1 "+5V" H 5800 4890 30  0000 C CNN
 F 2 "" H 5800 4800 60  0000 C CNN
@@
 	1    0    0    -1
 $EndComp
-Text GLabel 4450 2550 2    60   Input ~ 0
-REF+
-Text GLabel 4450 2750 2    60   Input ~ 0
-REF-
 $Comp
 L C C8
@@
 	3200 1550 3200 1900
 Wire Wire Line
-	4450 2550 4350 2550
-Wire Wire Line
-	4350 2550 4350 2600
+	4350 2400 4350 2600
 Wire Wire Line
 	4350 2600 4250 2600
@@
 	4250 2700 4350 2700
 Wire Wire Line
-	4350 2700 4350 2750
-Wire Wire Line
-	4350 2750 4450 2750
+	4350 2700 4350 2900
 Wire Wire Line
 	3300 1700 3200 1700
@@
 MISO
 $Comp
-L FE_V+ #PWR12
+L FE_V+ #PWR13
 U 1 1 5311A08F
 P 6750 3650
-F 0 "#PWR12" H 6750 3750 30  0001 C CNN
+F 0 "#PWR13" H 6750 3750 30  0001 C CNN
 F 1 "FE_V+" H 6750 3750 30  0000 C CNN
 F 2 "" H 6750 3650 60  0000 C CNN
@@
 $EndComp
 $Comp
-L FE_V+ #PWR16
+L FE_V+ #PWR17
 U 1 1 5311A095
 P 9200 4900
-F 0 "#PWR16" H 9200 5000 30  0001 C CNN
+F 0 "#PWR17" H 9200 5000 30  0001 C CNN
 F 1 "FE_V+" H 9200 5000 30  0000 C CNN
 F 2 "" H 9200 4900 60  0000 C CNN
@@
 $EndComp
 $Comp
-L FE_V+ #PWR13
+L FE_V+ #PWR14
 U 1 1 5311A09B
 P 9200 1700
-F 0 "#PWR13" H 9200 1800 30  0001 C CNN
+F 0 "#PWR14" H 9200 1800 30  0001 C CNN
 F 1 "FE_V+" H 9200 1800 30  0000 C CNN
 F 2 "" H 9200 1700 60  0000 C CNN
@@
 $EndComp
 $Comp
-L FE_V- #PWR15
+L FE_V- #PWR16
 U 1 1 5311A0A1
 P 9200 3900
-F 0 "#PWR15" H 9200 4100 40  0001 C CNN
+F 0 "#PWR16" H 9200 4100 40  0001 C CNN
 F 1 "FE_V-" H 9200 4050 40  0000 C CNN
 F 2 "~" H 9200 3900 60  0000 C CNN
@@
 $EndComp
 $Comp
-L FE_V- #PWR14
+L FE_V- #PWR15
 U 1 1 5311A0A7
 P 9200 2700
-F 0 "#PWR14" H 9200 2900 40  0001 C CNN
+F 0 "#PWR15" H 9200 2900 40  0001 C CNN
 F 1 "FE_V-" H 9200 2850 40  0000 C CNN
 F 2 "~" H 9200 2700 60  0000 C CNN
@@
 $EndComp
 $Comp
-L FE_V- #PWR11
+L FE_V- #PWR12
 U 1 1 5311A0AD
 P 6750 2600
-F 0 "#PWR11" H 6750 2800 40  0001 C CNN
+F 0 "#PWR12" H 6750 2800 40  0001 C CNN
 F 1 "FE_V-" H 6750 2750 40  0000 C CNN
 F 2 "~" H 6750 2600 60  0000 C CNN
@@
 $EndComp
 $Comp
-L AGND #PWR9
+L AGND #PWR10
 U 1 1 53137342
 P 6050 2750
-F 0 "#PWR9" H 6050 2750 40  0001 C CNN
+F 0 "#PWR10" H 6050 2750 40  0001 C CNN
 F 1 "AGND" H 6050 2680 50  0000 C CNN
 F 2 "" H 6050 2750 60  0000 C CNN
@@
 $EndComp
 $Comp
-L AGND #PWR10
+L AGND #PWR11
 U 1 1 53137352
 P 6050 3700
-F 0 "#PWR10" H 6050 3700 40  0001 C CNN
+F 0 "#PWR11" H 6050 3700 40  0001 C CNN
 F 1 "AGND" H 6050 3630 50  0000 C CNN
 F 2 "" H 6050 3700 60  0000 C CNN
@@
 $EndComp
 $Comp
-L AGND #PWR6
+L AGND #PWR7
 U 1 1 53137362
 P 5250 4550
-F 0 "#PWR6" H 5250 4550 40  0001 C CNN
+F 0 "#PWR7" H 5250 4550 40  0001 C CNN
 F 1 "AGND" H 5250 4480 50  0000 C CNN
 F 2 "" H 5250 4550 60  0000 C CNN
@@
 $EndComp
 $Comp
-L AGND #PWR7
+L AGND #PWR8
 U 1 1 53137372
 P 5250 6650
-F 0 "#PWR7" H 5250 6650 40  0001 C CNN
+F 0 "#PWR8" H 5250 6650 40  0001 C CNN
 F 1 "AGND" H 5250 6580 50  0000 C CNN
 F 2 "" H 5250 6650 60  0000 C CNN
@@
 	3150 1750 3200 1750
 Connection ~ 3200 1750
+$Comp
+L C C30
+U 1 1 53259593
+P 1250 2600
+F 0 "C30" H 1250 2700 40  0000 L CNN
+F 1 "C" H 1256 2515 40  0000 L CNN
+F 2 "SM0805" H 1288 2450 30  0000 C CNN
+F 3 "~" H 1250 2600 60  0000 C CNN
+	1    1250 2600
+	1    0    0    -1
+$EndComp
+Wire Wire Line
+	1250 2400 1250 2350
+Wire Wire Line
+	1250 2350 1550 2350
+Wire Wire Line
+	1550 2350 1550 2600
+Wire Wire Line
+	1550 2600 1600 2600
+Wire Wire Line
+	1600 2700 1550 2700
+Wire Wire Line
+	1550 2700 1550 2850
+Wire Wire Line
+	1550 2850 1250 2850
+Wire Wire Line
+	1250 2850 1250 2800
+$Comp
+L C C31
+U 1 1 532596D8
+P 4650 2650
+F 0 "C31" H 4650 2750 40  0000 L CNN
+F 1 "C" H 4656 2565 40  0000 L CNN
+F 2 "SM0805" H 4688 2500 30  0000 C CNN
+F 3 "~" H 4650 2650 60  0000 C CNN
+	1    4650 2650
+	1    0    0    -1
+$EndComp
+Wire Wire Line
+	4350 2400 4650 2400
+Wire Wire Line
+	4650 2400 4650 2450
+Wire Wire Line
+	4350 2900 4650 2900
+Wire Wire Line
+	4650 2900 4650 2850
+$Comp
+L AGND #PWR6
+U 1 1 532597F2
+P 4500 2950
+F 0 "#PWR6" H 4500 2950 40  0001 C CNN
+F 1 "AGND" H 4500 2880 50  0000 C CNN
+F 2 "" H 4500 2950 60  0000 C CNN
+F 3 "" H 4500 2950 60  0000 C CNN
+	1    4500 2950
+	1    0    0    -1
+$EndComp
+Wire Wire Line
+	4500 2950 4500 2900
+Connection ~ 4500 2900
 $EndSCHEMATC

Commit message: Layout Work Session 18
Parts:
- added TP1: 5V, symbol CONN_1
- added TP2: CH1+, symbol CONN_1
- added TP3: CH0+, symbol CONN_1
Connections:
- net +5V: now also TP1.1
- net CH0+: now also TP3.1
- net CH1+: now also TP2.1
Changed lines of the file:
@@
 Sheet 2 9
 Title ""
-Date "18 mar 2014"
+Date "20 mar 2014"
 Rev ""
 Comp ""
@@
 $EndComp
 $Comp
-L +5V #PWR01
+L +5V #PWR9
 U 1 1 5303ACCB
 P 5800 4800
-F 0 "#PWR01" H 5800 4890 20  0001 C CNN
+F 0 "#PWR9" H 5800 4890 20  0001 C CNN
 F 1 "+5V" H 5800 4890 30  0000 C CNN
 F 2 "" H 5800 4800 60  0000 C CNN
@@
 $EndComp
 $Comp
-L +5V #PWR02
+L +5V #PWR3
 U 1 1 5303B53D
 P 3200 1550
-F 0 "#PWR02" H 3200 1640 20  0001 C CNN
+F 0 "#PWR3" H 3200 1640 20  0001 C CNN
 F 1 "+5V" H 3200 1640 30  0000 C CNN
 F 2 "" H 3200 1550 60  0000 C CNN
@@
 	5600 2200 5250 2200
 Wire Wire Line
-	5250 2200 5250 3150
+	5250 1700 5250 3150
 Wire Wire Line
 	4250 3150 6150 3150
@@
 	4250 3600 4850 3600
 Wire Wire Line
-	4850 3600 4850 5600
+	4850 3400 4850 5600
 Wire Wire Line
 	4850 5600 5150 5600
@@
 MISO
 $Comp
-L FE_V+ #PWR03
+L FE_V+ #PWR13
 U 1 1 5311A08F
 P 6750 3650
-F 0 "#PWR03" H 6750 3750 30  0001 C CNN
+F 0 "#PWR13" H 6750 3750 30  0001 C CNN
 F 1 "FE_V+" H 6750 3750 30  0000 C CNN
 F 2 "" H 6750 3650 60  0000 C CNN
@@
 $EndComp
 $Comp
-L FE_V+ #PWR04
+L FE_V+ #PWR17
 U 1 1 5311A095
 P 9200 4900
-F 0 "#PWR04" H 9200 5000 30  0001 C CNN
+F 0 "#PWR17" H 9200 5000 30  0001 C CNN
 F 1 "FE_V+" H 9200 5000 30  0000 C CNN
 F 2 "" H 9200 4900 60  0000 C CNN
@@
 $EndComp
 $Comp
-L FE_V+ #PWR05
+L FE_V+ #PWR14
 U 1 1 5311A09B
 P 9200 1700
-F 0 "#PWR05" H 9200 1800 30  0001 C CNN
+F 0 "#PWR14" H 9200 1800 30  0001 C CNN
 F 1 "FE_V+" H 9200 1800 30  0000 C CNN
 F 2 "" H 9200 1700 60  0000 C CNN
@@
 $EndComp
 $Comp
-L AGND #PWR06
+L AGND #PWR2
 U 1 1 5313730A
 P 2650 4550
-F 0 "#PWR06" H 2650 4550 40  0001 C CNN
+F 0 "#PWR2" H 2650 4550 40  0001 C CNN
 F 1 "AGND" H 2650 4480 50  0000 C CNN
 F 2 "" H 2650 4550 60  0000 C CNN
@@
 $EndComp
 $Comp
-L AGND #PWR07
+L AGND #PWR4
 U 1 1 53137321
 P 3200 4550
-F 0 "#PWR07" H 3200 4550 40  0001 C CNN
+F 0 "#PWR4" H 3200 4550 40  0001 C CNN
 F 1 "AGND" H 3200 4480 50  0000 C CNN
 F 2 "" H 3200 4550 60  0000 C CNN
@@
 $EndComp
 $Comp
-L AGND #PWR08
+L AGND #PWR1
 U 1 1 5313732C
 P 1700 1800
-F 0 "#PWR08" H 1700 1800 40  0001 C CNN
+F 0 "#PWR1" H 1700 1800 40  0001 C CNN
 F 1 "AGND" H 1700 1730 50  0000 C CNN
 F 2 "" H 1700 1800 60  0000 C CNN
@@
 $EndComp
 $Comp
-L AGND #PWR09
+L AGND #PWR5
 U 1 1 5313733C
 P 3850 1800
-F 0 "#PWR09" H 3850 1800 40  0001 C CNN
+F 0 "#PWR5" H 3850 1800 40  0001 C CNN
 F 1 "AGND" H 3850 1730 50  0000 C CNN
 F 2 "" H 3850 1800 60  0000 C CNN
@@
 $EndComp
 $Comp
-L AGND #PWR010
+L AGND #PWR10
 U 1 1 53137342
 P 6050 2750
-F 0 "#PWR010" H 6050 2750 40  0001 C CNN
+F 0 "#PWR10" H 6050 2750 40  0001 C CNN
 F 1 "AGND" H 6050 2680 50  0000 C CNN
 F 2 "" H 6050 2750 60  0000 C CNN
@@
 $EndComp
 $Comp
-L AGND #PWR011
+L AGND #PWR11
 U 1 1 53137352
 P 6050 3700
-F 0 "#PWR011" H 6050 3700 40  0001 C CNN
+F 0 "#PWR11" H 6050 3700 40  0001 C CNN
 F 1 "AGND" H 6050 3630 50  0000 C CNN
 F 2 "" H 6050 3700 60  0000 C CNN
@@
 $EndComp
 $Comp
-L AGND #PWR012
+L AGND #PWR7
 U 1 1 53137362
 P 5250 4550
-F 0 "#PWR012" H 5250 4550 40  0001 C CNN
+F 0 "#PWR7" H 5250 4550 40  0001 C CNN
 F 1 "AGND" H 5250 4480 50  0000 C CNN
 F 2 "" H 5250 4550 60  0000 C CNN
@@
 $EndComp
 $Comp
-L AGND #PWR013
+L AGND #PWR8
 U 1 1 53137372
 P 5250 6650
-F 0 "#PWR013" H 5250 6650 40  0001 C CNN
+F 0 "#PWR8" H 5250 6650 40  0001 C CNN
 F 1 "AGND" H 5250 6580 50  0000 C CNN
 F 2 "" H 5250 6650 60  0000 C CNN
@@
 	4650 2900 4650 2850
 $Comp
-L AGND #PWR014
+L AGND #PWR6
 U 1 1 532597F2
 P 4500 2950
-F 0 "#PWR014" H 4500 2950 40  0001 C CNN
+F 0 "#PWR6" H 4500 2950 40  0001 C CNN
 F 1 "AGND" H 4500 2880 50  0000 C CNN
 F 2 "" H 4500 2950 60  0000 C CNN
@@
 	4500 2950 4500 2900
 Connection ~ 4500 2900
+$Comp
+L CONN_1 TP3
+U 1 1 532B3628
+P 5400 1700
+F 0 "TP3" H 5480 1700 40  0000 L CNN
+F 1 "CH0+" H 5400 1755 30  0001 C CNN
+F 2 "" H 5400 1700 60  0000 C CNN
+F 3 "" H 5400 1700 60  0000 C CNN
+	1    5400 1700
+	1    0    0    -1
+$EndComp
+Connection ~ 5250 2200
+$Comp
+L CONN_1 TP2
+U 1 1 532B36E1
+P 4600 3400
+F 0 "TP2" H 4680 3400 40  0000 L CNN
+F 1 "CH1+" H 4600 3455 30  0001 C CNN
+F 2 "" H 4600 3400 60  0000 C CNN
+F 3 "" H 4600 3400 60  0000 C CNN
+	1    4600 3400
+	-1   0    0    1
+$EndComp
+Wire Wire Line
+	4750 3400 4850 3400
+Connection ~ 4850 3600
+$Comp
+L CONN_1 TP1
+U 1 1 532B578B
+P 3500 1550
+F 0 "TP1" H 3580 1550 40  0000 L CNN
+F 1 "5V" H 3500 1605 30  0001 C CNN
+F 2 "" H 3500 1550 60  0000 C CNN
+F 3 "" H 3500 1550 60  0000 C CNN
+	1    3500 1550
+	1    0    0    -1
+$EndComp
+Wire Wire Line
+	3350 1550 3300 1550
+Wire Wire Line
+	3300 1550 3300 1600
+Wire Wire Line
+	3300 1600 3200 1600
+Connection ~ 3200 1600
 $EndSCHEMATC
