File: BenchBudEE/Relay.sch (KiCad schematic (older format))
At the start: 11 parts, among them K1 1461069-5, Q1 2N3904, U1 LTV-816S

Commit message: Reality Check
Connections:
- net RELAY_NC: now also K1.3 (NO); no longer K1.4 (NC)
- net RELAY_NO: now also K1.4 (NC); no longer K1.3 (NO)
Changed lines of the file:
@@
 Text HLabel 2950 3350 0    60   Output ~ 0
 RELAY-
+Text HLabel 10050 2750 2    60   BiDi ~ 0
+RELAY_NC
 Text HLabel 10050 2550 2    60   BiDi ~ 0
-RELAY_NC
-Text HLabel 10050 2750 2    60   BiDi ~ 0
 RELAY_NO
 $Comp

Commit message: Layout Work Session 4
Connections:
- net GND renamed GND_RELAY
Changed lines of the file:
@@
 Sheet 5 9
 Title ""
-Date "1 mar 2014"
+Date "2 mar 2014"
 Rev ""
 Comp ""
@@
 Wire Wire Line
 	8300 4550 8300 4800
-$Comp
-L GND #PWR032
-U 1 1 52F62F52
-P 8300 4800
-F 0 "#PWR032" H 8300 4800 30  0001 C CNN
-F 1 "GND" H 8300 4730 30  0001 C CNN
-F 2 "" H 8300 4800 60  0000 C CNN
-F 3 "" H 8300 4800 60  0000 C CNN
-	1    8300 4800
-	1    0    0    -1
-$EndComp
 Wire Wire Line
 	6300 3350 6300 3500
@@
 	6500 1700 6500 1350
 $Comp
-L +12P #PWR033
+L +12P #PWR032
 U 1 1 52F63026
 P 6500 1350
-F 0 "#PWR033" H 6500 1320 30  0001 C CNN
+F 0 "#PWR032" H 6500 1320 30  0001 C CNN
 F 1 "+12P" H 6500 1450 30  0000 C CNN
 F 2 "" H 6500 1350 60  0000 C CNN
@@
 	7650 1400 6500 1400
 Connection ~ 6500 1400
+$Comp
+L GND_RELAY #PWR033
+U 1 1 53133457
+P 8300 4800
+F 0 "#PWR033" H 8300 4800 30  0001 C CNN
+F 1 "GND_RELAY" H 8300 4730 30  0000 C CNN
+F 2 "" H 8300 4800 60  0000 C CNN
+F 3 "" H 8300 4800 60  0000 C CNN
+	1    8300 4800
+	1    0    0    -1
+$EndComp
 $EndSCHEMATC
