File: BenchBudEE/Power.sch (KiCad schematic (older format))
At the start: 13 parts, among them P1 24 pin Mini-fit Jr, SW1 Power Switch

Commit message: Layout Work Session 5
Parts:
- added TP1: CONN_1, symbol CONN_1
Connections:
- net GND: now also TP1.1
Changed lines of the file:
@@
 	3500 1850 3500 1350
 Connection ~ 3500 1350
+$Comp
+L CONN_1 TP1
+U 1 1 531391A7
+P 6800 2800
+F 0 "TP1" H 6880 2800 40  0000 L CNN
+F 1 "CONN_1" H 6800 2855 30  0001 C CNN
+F 2 "" H 6800 2800 60  0000 C CNN
+F 3 "" H 6800 2800 60  0000 C CNN
+	1    6800 2800
+	-1   0    0    1
+$EndComp
+$Comp
+L GND #PWR032
+U 1 1 531391B4
+P 7050 2900
+F 0 "#PWR032" H 7050 2900 30  0001 C CNN
+F 1 "GND" H 7050 2830 30  0001 C CNN
+F 2 "" H 7050 2900 60  0000 C CNN
+F 3 "" H 7050 2900 60  0000 C CNN
+	1    7050 2900
+	1    0    0    -1
+$EndComp
+Wire Wire Line
+	6950 2800 7050 2800
+Wire Wire Line
+	7050 2800 7050 2900
 $EndSCHEMATC

Commit message: Layout Work Session 6
Parts:
- added JP1, JP2, JP3, JP4: JUMPER, ~, symbol JUMPER
Connections:
- net GND: now also JP1.1, JP2.1, JP3.1, JP4.1
- new net AGND: JP1.2
- new net GND_LED: JP3.2
- new net GND_PWR: JP2.2
- new net GND_RELAY: JP4.2
Other:
- note added: "Star Point"
- moved on the sheet: TP1
Changed lines of the file:
@@
 Sheet 4 9
 Title ""
-Date "2 mar 2014"
+Date "3 mar 2014"
 Rev ""
 Comp ""
@@
 	1700 1450 1700 1600
 $Comp
-L GND #PWR018
+L GND #PWR22
 U 1 1 52F65191
 P 1700 1600
-F 0 "#PWR018" H 1700 1600 30  0001 C CNN
+F 0 "#PWR22" H 1700 1600 30  0001 C CNN
 F 1 "GND" H 1700 1530 30  0001 C CNN
 F 2 "" H 1700 1600 60  0000 C CNN
@@
 	3100 1950 5900 1950
 $Comp
-L +12P #PWR019
+L +12P #PWR34
 U 1 1 52F65291
 P 5850 1000
-F 0 "#PWR019" H 5850 970 30  0001 C CNN
+F 0 "#PWR34" H 5850 970 30  0001 C CNN
 F 1 "+12P" H 5850 1100 30  0000 C CNN
 F 2 "" H 5850 1000 60  0000 C CNN
@@
 	5850 1750 5650 1750
 $Comp
-L -12P #PWR020
+L -12P #PWR35
 U 1 1 52F65D56
 P 6600 1000
-F 0 "#PWR020" H 6600 1130 20  0001 C CNN
+F 0 "#PWR35" H 6600 1130 20  0001 C CNN
 F 1 "-12P" H 6600 1100 30  0000 C CNN
 F 2 "" H 6600 1000 60  0000 C CNN
@@
 $EndComp
 $Comp
-L GND #PWR021
+L GND #PWR26
 U 1 1 52F65E0B
 P 4700 3200
-F 0 "#PWR021" H 4700 3200 30  0001 C CNN
+F 0 "#PWR26" H 4700 3200 30  0001 C CNN
 F 1 "GND" H 4700 3130 30  0001 C CNN
 F 2 "" H 4700 3200 60  0000 C CNN
@@
 	5600 2800 5600 2400
 $Comp
-L +3.3V #PWR022
+L +3.3V #PWR32
 U 1 1 52F66046
 P 5600 2400
-F 0 "#PWR022" H 5600 2360 30  0001 C CNN
+F 0 "#PWR32" H 5600 2360 30  0001 C CNN
 F 1 "+3.3V" H 5600 2510 30  0000 C CNN
 F 2 "" H 5600 2400 60  0000 C CNN
@@
 $EndComp
 $Comp
-L -12P #PWR023
+L -12P #PWR37
 U 1 1 52F6604C
 P 8050 3000
-F 0 "#PWR023" H 8050 3130 20  0001 C CNN
+F 0 "#PWR37" H 8050 3130 20  0001 C CNN
 F 1 "-12P" H 8050 3100 30  0000 C CNN
 F 2 "" H 8050 3000 60  0000 C CNN
@@
 $EndComp
 $Comp
-L +12P #PWR024
+L +12P #PWR36
 U 1 1 52F66052
 P 8050 1900
-F 0 "#PWR024" H 8050 1870 30  0001 C CNN
+F 0 "#PWR36" H 8050 1870 30  0001 C CNN
 F 1 "+12P" H 8050 2000 30  0000 C CNN
 F 2 "" H 8050 1900 60  0000 C CNN
@@
 Connection ~ 9250 2450
 $Comp
-L GND #PWR025
+L GND #PWR39
 U 1 1 52F6614F
 P 8700 2550
-F 0 "#PWR025" H 8700 2550 30  0001 C CNN
+F 0 "#PWR39" H 8700 2550 30  0001 C CNN
 F 1 "GND" H 8700 2480 30  0001 C CNN
 F 2 "" H 8700 2550 60  0000 C CNN
@@
 Connection ~ 9250 1950
 $Comp
-L +12V #PWR026
+L +12V #PWR41
 U 1 1 52F661D8
 P 9800 1900
-F 0 "#PWR026" H 9800 1850 20  0001 C CNN
+F 0 "#PWR41" H 9800 1850 20  0001 C CNN
 F 1 "+12V" H 9800 2000 30  0000 C CNN
 F 2 "" H 9800 1900 60  0000 C CNN
@@
 $EndComp
 $Comp
-L -12V #PWR027
+L -12V #PWR42
 U 1 1 52F661F1
 P 9800 3000
-F 0 "#PWR027" H 9800 3130 20  0001 C CNN
+F 0 "#PWR42" H 9800 3130 20  0001 C CNN
 F 1 "-12V" H 9800 3100 30  0000 C CNN
 F 2 "" H 9800 3000 60  0000 C CNN
@@
 Connection ~ 3400 1750
 $Comp
-L +12C #PWR028
+L +12C #PWR23
 U 1 1 52FA733D
 P 3400 1000
-F 0 "#PWR028" H 3400 970 30  0001 C CNN
+F 0 "#PWR23" H 3400 970 30  0001 C CNN
 F 1 "+12C" H 3400 1110 40  0000 C CNN
 F 2 "" H 3400 1000 60  0000 C CNN
@@
 	9100 800  9850 800
 $Comp
-L GND #PWR029
+L GND #PWR40
 U 1 1 5300ADC6
 P 9300 1400
-F 0 "#PWR029" H 9300 1400 30  0001 C CNN
+F 0 "#PWR40" H 9300 1400 30  0001 C CNN
 F 1 "GND" H 9300 1330 30  0001 C CNN
 F 2 "" H 9300 1400 60  0000 C CNN
@@
 Connection ~ 9300 800
 $Comp
-L +5P #PWR26
+L +5P #PWR27
 U 1 1 5300AE45
 P 5000 1000
-F 0 "#PWR26" H 5000 1130 20  0001 C CNN
+F 0 "#PWR27" H 5000 1130 20  0001 C CNN
 F 1 "+5P" H 5000 1100 30  0000 C CNN
 F 2 "" H 5000 1000 60  0000 C CNN
@@
 $EndComp
 $Comp
-L +5P #PWR32
+L +5P #PWR38
 U 1 1 5300AE61
 P 8100 750
-F 0 "#PWR32" H 8100 880 20  0001 C CNN
+F 0 "#PWR38" H 8100 880 20  0001 C CNN
 F 1 "+5P" H 8100 850 30  0000 C CNN
 F 2 "" H 8100 750 60  0000 C CNN
@@
 $EndComp
 $Comp
-L +5V #PWR030
+L +5V #PWR43
 U 1 1 5300AE69
 P 9850 750
-F 0 "#PWR030" H 9850 840 20  0001 C CNN
+F 0 "#PWR43" H 9850 840 20  0001 C CNN
 F 1 "+5V" H 9850 840 30  0000 C CNN
 F 2 "" H 9850 750 60  0000 C CNN
@@
 	9300 1250 9300 1400
 $Comp
-L +3.3V #PWR031
+L +3.3V #PWR25
 U 1 1 5311B0C2
 P 4350 1000
-F 0 "#PWR031" H 4350 960 30  0001 C CNN
+F 0 "#PWR25" H 4350 960 30  0001 C CNN
 F 1 "+3.3V" H 4350 1110 30  0000 C CNN
 F 2 "" H 4350 1000 60  0000 C CNN
@@
 L CONN_1 TP1
 U 1 1 531391A7
-P 6800 2800
-F 0 "TP1" H 6880 2800 40  0000 L CNN
-F 1 "CONN_1" H 6800 2855 30  0001 C CNN
-F 2 "" H 6800 2800 60  0000 C CNN
-F 3 "" H 6800 2800 60  0000 C CNN
-	1    6800 2800
+P 5350 5050
+F 0 "TP1" H 5430 5050 40  0000 L CNN
+F 1 "CONN_1" H 5350 5105 30  0001 C CNN
+F 2 "" H 5350 5050 60  0000 C CNN
+F 3 "" H 5350 5050 60  0000 C CNN
+	1    5350 5050
 	-1   0    0    1
 $EndComp
 $Comp
-L GND #PWR032
+L GND #PWR33
 U 1 1 531391B4
-P 7050 2900
-F 0 "#PWR032" H 7050 2900 30  0001 C CNN
-F 1 "GND" H 7050 2830 30  0001 C CNN
-F 2 "" H 7050 2900 60  0000 C CNN
-F 3 "" H 7050 2900 60  0000 C CNN
-	1    7050 2900
-	1    0    0    -1
-$EndComp
-Wire Wire Line
-	6950 2800 7050 2800
-Wire Wire Line
-	7050 2800 7050 2900
+P 5600 5150
+F 0 "#PWR33" H 5600 5150 30  0001 C CNN
+F 1 "GND" H 5600 5080 30  0001 C CNN
+F 2 "" H 5600 5150 60  0000 C CNN
+F 3 "" H 5600 5150 60  0000 C CNN
+	1    5600 5150
+	1    0    0    -1
+$EndComp
+Wire Wire Line
+	5500 5050 5600 5050
+Wire Wire Line
+	5600 5050 5600 5150
+$Comp
+L JUMPER JP1
+U 1 1 5314DDDA
+P 4700 5500
+F 0 "JP1" H 4700 5650 60  0000 C CNN
+F 1 "JUMPER" H 4700 5420 40  0000 C CNN
+F 2 "~" H 4700 5500 60  0000 C CNN
+F 3 "~" H 4700 5500 60  0000 C CNN
+	1    4700 5500
+	1    0    0    -1
+$EndComp
+Text Notes 5150 4900 0    60   ~ 0
+Star Point
+$Comp
+L JUMPER JP2
+U 1 1 5314DDF1
+P 4700 5850
+F 0 "JP2" H 4700 6000 60  0000 C CNN
+F 1 "JUMPER" H 4700 5770 40  0000 C CNN
+F 2 "~" H 4700 5850 60  0000 C CNN
+F 3 "~" H 4700 5850 60  0000 C CNN
+	1    4700 5850
+	1    0    0    -1
+$EndComp
+$Comp
+L JUMPER JP3
+U 1 1 5314DDF7
+P 4700 6250
+F 0 "JP3" H 4700 6400 60  0000 C CNN
+F 1 "JUMPER" H 4700 6170 40  0000 C CNN
+F 2 "~" H 4700 6250 60  0000 C CNN
+F 3 "~" H 4700 6250 60  0000 C CNN
+	1    4700 6250
+	1    0    0    -1
+$EndComp
+$Comp
+L JUMPER JP4
+U 1 1 5314DDFD
+P 4700 6650
+F 0 "JP4" H 4700 6800 60  0000 C CNN
+F 1 "JUMPER" H 4700 6570 40  0000 C CNN
+F 2 "~" H 4700 6650 60  0000 C CNN
+F 3 "~" H 4700 6650 60  0000 C CNN
+	1    4700 6650
+	1    0    0    -1
+$EndComp
+$Comp
+L GND #PWR24
+U 1 1 5314DE30
+P 4250 6850
+F 0 "#PWR24" H 4250 6850 30  0001 C CNN
+F 1 "GND" H 4250 6780 30  0001 C CNN
+F 2 "" H 4250 6850 60  0000 C CNN
+F 3 "" H 4250 6850 60  0000 C CNN
+	1    4250 6850
+	1    0    0    -1
+$EndComp
+Wire Wire Line
+	4250 6850 4250 5500
+Wire Wire Line
+	4250 5500 4400 5500
+Wire Wire Line
+	4400 5850 4250 5850
+Connection ~ 4250 5850
+Wire Wire Line
+	4400 6250 4250 6250
+Connection ~ 4250 6250
+Wire Wire Line
+	4400 6650 4250 6650
+Connection ~ 4250 6650
+$Comp
+L GND_LED #PWR30
+U 1 1 5314DF91
+P 5150 6350
+F 0 "#PWR30" H 5150 6350 30  0001 C CNN
+F 1 "GND_LED" H 5150 6280 30  0000 C CNN
+F 2 "~" H 5150 6350 60  0000 C CNN
+F 3 "~" H 5150 6350 60  0000 C CNN
+	1    5150 6350
+	1    0    0    -1
+$EndComp
+$Comp
+L GND_PWR #PWR29
+U 1 1 5314DFA0
+P 5150 5950
+F 0 "#PWR29" H 5150 5950 30  0001 C CNN
+F 1 "GND_PWR" H 5150 5880 30  0000 C CNN
+F 2 "~" H 5150 5950 60  0000 C CNN
+F 3 "~" H 5150 5950 60  0000 C CNN
+	1    5150 5950
+	1    0    0    -1
+$EndComp
+$Comp
+L GND_RELAY #PWR31
+U 1 1 5314DFAF
+P 5150 6750
+F 0 "#PWR31" H 5150 6750 30  0001 C CNN
+F 1 "GND_RELAY" H 5150 6680 30  0000 C CNN
+F 2 "~" H 5150 6750 60  0000 C CNN
+F 3 "~" H 5150 6750 60  0000 C CNN
+	1    5150 6750
+	1    0    0    -1
+$EndComp
+$Comp
+L AGND #PWR28
+U 1 1 5314DFBE
+P 5150 5600
+F 0 "#PWR28" H 5150 5600 40  0001 C CNN
+F 1 "AGND" H 5150 5530 50  0000 C CNN
+F 2 "~" H 5150 5600 60  0000 C CNN
+F 3 "~" H 5150 5600 60  0000 C CNN
+	1    5150 5600
+	1    0    0    -1
+$EndComp
+Wire Wire Line
+	5000 5500 5150 5500
+Wire Wire Line
+	5150 5500 5150 5600
+Wire Wire Line
+	5000 5850 5150 5850
+Wire Wire Line
+	5150 5850 5150 5950
+Wire Wire Line
+	5000 6250 5150 6250
+Wire Wire Line
+	5150 6250 5150 6350
+Wire Wire Line
+	5000 6650 5150 6650
+Wire Wire Line
+	5150 6650 5150 6750
 $EndSCHEMATC
