File: BenchBudEE/LED_Driver.sch (KiCad schematic (older format))
At the start: 6 parts, among them U5 AP5726

Commit message: Layout Work Session 4
Connections:
- net GND renamed GND_LED
Changed lines of the file:
@@
 Sheet 3 9
 Title ""
-Date "1 mar 2014"
+Date "2 mar 2014"
 Rev ""
 Comp ""
@@
 F 3 "" H 3200 2050 60  0000 C CNN
 	1    3300 2150
-	1    0    0    -1
-$EndComp
-$Comp
-L GND #PWR015
-U 1 1 52F7B18F
-P 2250 1750
-F 0 "#PWR015" H 2250 1750 30  0001 C CNN
-F 1 "GND" H 2250 1680 30  0001 C CNN
-F 2 "" H 2250 1750 60  0000 C CNN
-F 3 "" H 2250 1750 60  0000 C CNN
-	1    2250 1750
-	1    0    0    -1
-$EndComp
-$Comp
-L GND #PWR016
-U 1 1 52F7B19C
-P 3250 3000
-F 0 "#PWR016" H 3250 3000 30  0001 C CNN
-F 1 "GND" H 3250 2930 30  0001 C CNN
-F 2 "" H 3250 3000 60  0000 C CNN
-F 3 "" H 3250 3000 60  0000 C CNN
-	1    3250 3000
 	1    0    0    -1
 $EndComp
@@
 	8850 1150 8850 1200
 Connection ~ 4050 1150
-$Comp
-L GND #PWR017
-U 1 1 52F7B218
-P 8850 1700
-F 0 "#PWR017" H 8850 1700 30  0001 C CNN
-F 1 "GND" H 8850 1630 30  0001 C CNN
-F 2 "" H 8850 1700 60  0000 C CNN
-F 3 "" H 8850 1700 60  0000 C CNN
-	1    8850 1700
-	1    0    0    -1
-$EndComp
 Wire Wire Line
 	8850 1600 8850 1700
@@
 	1    0    0    -1
 $EndComp
+$Comp
+L GND_LED #PWR015
+U 1 1 53132E60
+P 3250 3000
+F 0 "#PWR015" H 3250 3000 30  0001 C CNN
+F 1 "GND_LED" H 3250 2930 30  0000 C CNN
+F 2 "" H 3250 3000 60  0000 C CNN
+F 3 "" H 3250 3000 60  0000 C CNN
+	1    3250 3000
+	1    0    0    -1
+$EndComp
+$Comp
+L GND_LED #PWR016
+U 1 1 53132E72
+P 2250 1750
+F 0 "#PWR016" H 2250 1750 30  0001 C CNN
+F 1 "GND_LED" H 2250 1680 30  0000 C CNN
+F 2 "" H 2250 1750 60  0000 C CNN
+F 3 "" H 2250 1750 60  0000 C CNN
+	1    2250 1750
+	1    0    0    -1
+$EndComp
+$Comp
+L GND_LED #PWR017
+U 1 1 53132E78
+P 8850 1700
+F 0 "#PWR017" H 8850 1700 30  0001 C CNN
+F 1 "GND_LED" H 8850 1630 30  0000 C CNN
+F 2 "" H 8850 1700 60  0000 C CNN
+F 3 "" H 8850 1700 60  0000 C CNN
+	1    8850 1700
+	1    0    0    -1
+$EndComp
